Commit message: chore: add intertial and collision to gripper

File: src/kinova_description/urdf/kinova.urdf (robot description, URDF)
Before this commit: robot kinova_arm, 11 links, 10 joints
Links:
- link GRIPPER_FRAME: mass None -> 0.1395; geometry collision mesh filename=package://kinova_description/meshes/gripper_base_link.STL; visual mesh filename=package://kinova_description/meshes/gripper_base_link.STL
- link LEFT_FINGER_DIST: mass None -> 0.010748; geometry collision mesh filename=package://kinova_description/meshes/left_finger_dist_link.S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; visual mesh filename=package://kinova_description/meshes/left_finger_dist_link.S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
- link LEFT_FINGER_PROX: mass None -> 0.018385; geometry collision mesh filename=package://kinova_description/meshes/left_finger_prox_link.S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; visual mesh filename=package://kinova_description/meshes/left_finger_prox_link.S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
- link RIGHT_FINGER_DIST: mass None -> 0.010748; geometry collision mesh filename=package://kinova_description/meshes/right_finger_dist_link.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; visual mesh filename=package://kinova_description/meshes/right_finger_dist_link.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
- link RIGHT_FINGER_PROX: mass None -> 0.018385; geometry collision mesh filename=package://kinova_description/meshes/right_finger_prox_link.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; visual mesh filename=package://kinova_description/meshes/right_finger_prox_link.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

Commit message: fix: modify left_bottom max limit for perfect grip close

File: src/kinova_description/urdf/kinova.urdf (robot description, URDF)
Before this commit: robot kinova_arm, 11 links, 10 joints
Joints:
- joint LEFT_BOTTOM: limit lower=-0.96 upper=0.09 effort=1000 velocity=1000 -> lower=-0.96 upper=0.22 effort=1000 velocity=1000
